File: pcb/template.kicad_sch (KiCad schematic)
At the start: 0 parts

Commit message: Tweaking KiCAD template...
Other:
- title: Ear Tag -> Top Level
Changed lines of the file:
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@@
   (paper "A3")
   (title_block
-    (title "Ear Tag")
-    (date "2023-09-03")
+    (title "Top Level")
+    (date "2024-02-29")
     (rev "0.1")
   )
